File: PCB kiCAD/flight controller.sch (KiCad schematic (older format))
At the start: 28 parts, among them J1 ESC3, J2 ESC4, J3 LED4, J4 LED3, J5 LED1, J6 ESC1, J7 LED2, J8 ESC2, J9 Lidar, U1 YAAJ_BluePill_Part_Like, U2 mpu6050pcb, U3 FTDI, U4 gps, U5 gps, U6 Barometer, U7 mpu6050pcb

Commit message: fix schematic png
Parts:
- D1, D2, D3, D4: footprint (none) -> LED_THT:LED_D4.0mm
- J1, J2, J6, J8: footprint (none) -> Connector_PinHeader_2.54mm:PinHeader_1x03_P2.54mm_Horizontal
- J10: renamed from J?; footprint (none) -> Connector_PinHeader_2.54mm:PinHeader_1x03_P2.54mm_Horizontal
- J11: renamed from J?; footprint (none) -> Connector_PinHeader_2.54mm:PinHeader_1x01_P2.54mm_Horizontal
- J3, J4, J5, J7: footprint (none) -> Connector_PinHeader_2.54mm:PinHeader_1x02_P2.54mm_Horizontal
- J9: footprint (none) -> Connector_PinHeader_2.54mm:PinHeader_1x04_P2.54mm_Horizontal
- R1, R2, R3, R4: footprint (none) -> Resistor_THT:R_Axial_DIN0411_L9.9mm_D3.6mm_P12.70mm_Horizontal
- R5, R6: renamed from R?; footprint (none) -> Resistor_THT:R_Axial_DIN0411_L9.9mm_D3.6mm_P12.70mm_Horizontal
- U1: footprint (none) -> Drone:YAAJ_BluePill_1
- U2, U7: footprint (none) -> Footprints:IMU
- U3: footprint (none) -> Socket_Strips:Socket_Strip_Angled_1x06_Pitch2.54mm
- U4, U5: footprint (none) -> Footprints:GPS
- U6: footprint (none) -> Footprints:Barometer
Connections:
- wire segments 99 -> 100
- no-connect marks 28 -> 27
Other:
- moved on the sheet: J10, J2, J3, J9

Commit message: ny pcb
Connections:
- wire segments 100 -> 102
Changed lines of the file:
@@
 Text Label 4650 1600 0    50   ~ 0
 ESC1
+Text Label 7700 1800 2    50   ~ 0
+SDA
+Wire Wire Line
+	7700 1800 7900 1800
 Text Label 7700 2000 2    50   ~ 0
-SDA
+SCL
 Wire Wire Line
 	7700 2000 7900 2000
-Text Label 7700 1800 2    50   ~ 0
-SCL
-Wire Wire Line
-	7700 1800 7900 1800
 $Comp
 L gps:gps U4
@@
 $EndComp
 Wire Wire Line
+	8800 2000 8600 2000
+Wire Wire Line
 	8800 1800 8600 1800
-Wire Wire Line
-	8800 2000 8600 2000
 Wire Notes Line
 	7000 3400 5500 3400
@@
 L power:Earth #PWR0113
 U 1 1 61AE4ACD
-P 8600 3400
-F 0 "#PWR0113" H 8600 3150 50  0001 C CNN
-F 1 "Earth" H 8600 3250 50  0001 C CNN
-F 2 "" H 8600 3400 50  0001 C CNN
-F 3 "~" H 8600 3400 50  0001 C CNN
-	1    8600 3400
+P 8750 2800
+F 0 "#PWR0113" H 8750 2550 50  0001 C CNN
+F 1 "Earth" H 8750 2650 50  0001 C CNN
+F 2 "" H 8750 2800 50  0001 C CNN
+F 3 "~" H 8750 2800 50  0001 C CNN
+	1    8750 2800
 	1    0    0    -1
 $EndComp
@@
 5V
 Wire Wire Line
+	8800 3000 8600 3000
+Wire Wire Line
 	8800 3200 8600 3200
-Wire Wire Line
-	8800 3000 8600 3000
+Text Label 8800 3200 0    50   ~ 0
+RX
 Text Label 8800 3000 0    50   ~ 0
-RX
-Text Label 8800 3200 0    50   ~ 0
 TX
 Wire Wire Line
-	8800 2800 8600 2800
-Text Label 8800 2800 0    50   ~ 0
+	8800 3400 8600 3400
+Text Label 8800 3400 0    50   ~ 0
 5V
 Wire Wire Line
-	8800 1600 8600 1600
-Text Label 8800 1600 0    50   ~ 0
+	8800 2200 8600 2200
+Text Label 8800 2200 0    50   ~ 0
 5V
+Text Label 8800 2000 0    50   ~ 0
+RX2
 Text Label 8800 1800 0    50   ~ 0
-RX2
-Text Label 8800 2000 0    50   ~ 0
 TX2
 $Comp
 L power:Earth #PWR0106
 U 1 1 61A90FD5
-P 8600 2200
-F 0 "#PWR0106" H 8600 1950 50  0001 C CNN
-F 1 "Earth" H 8600 2050 50  0001 C CNN
-F 2 "" H 8600 2200 50  0001 C CNN
-F 3 "~" H 8600 2200 50  0001 C CNN
-	1    8600 2200
+P 8800 1600
+F 0 "#PWR0106" H 8800 1350 50  0001 C CNN
+F 1 "Earth" H 8800 1450 50  0001 C CNN
+F 2 "" H 8800 1600 50  0001 C CNN
+F 3 "~" H 8800 1600 50  0001 C CNN
+	1    8800 1600
 	1    0    0    -1
 $EndComp
@@
 Wire Wire Line
 	8650 4600 8800 4600
+Wire Wire Line
+	8800 1600 8600 1600
+Wire Wire Line
+	8750 2800 8600 2800
 $EndSCHEMATC
